Commit message: Multi robot, collision, senors. What mus be revised colision while sliding over walls it glitches in the map generated by the sensors and rviz.

File: src/khepera4_description/urdf/khepera4.urdf (robot description, URDF)
Before this commit: robot khepera4, 26 links, 25 joints
Links:
- link base_link: geometry collision cylinder length=0.0095 radius=0.050; collision cylinder length=0.044 radius=0.070
